File: SL40.kicad_pcb (KiCad board)
At the start: 2 copper layers, 266.7 x 76.2 mm, 99 parts, among them SW1 SW_Push, U1 Arduino Pro Micro

Commit message: adding new layouts
Parts:
- added  : 2.25U, MX_Alps_Hybrid:MX-2.25U-ReversedStabilizers-NoLED, F.Cu at (259.6, 100.8)
- added  : 1U, MX_Alps_Hybrid:MX-1U-NoLED, F.Cu at (228.6, 100.8)
- added  : 1U, MX_Alps_Hybrid:MX-1U-NoLED, F.Cu at (247.7, 100.8)
- added  : 1.25U, MX_Alps_Hybrid:MX-1.25U-NoLED, F.Cu at (269.1, 100.8)
- added  : 2U, MX_Alps_Hybrid:MX-2U-ReversedStabilizers-NoLED, F.Cu at (166.7, 119.9)
- added  : 2.25U, MX_Alps_Hybrid:MX-2.25U-ReversedStabilizers-NoLED, F.Cu at (126.2, 119.9)
- added  : 1U, MX_Alps_Hybrid:MX-1U-NoLED, F.Cu at (95.2, 119.9)
- added  : 1U, MX_Alps_Hybrid:MX-1U-NoLED, F.Cu at (195.3, 119.9)
- added  : 2U, MX_Alps_Hybrid:MX-2U-NoLED, F.Cu at (261.9, 62.7)
- added D1: D_small, combodiode:ComboDiode, F.Cu at (103.2, 119.1)
- added D1: D_small, combodiode:ComboDiode, F.Cu at (134.1, 119.9)
- added D1: D_small, combodiode:ComboDiode, F.Cu at (174.6, 119.9)
- added D1: D_small, combodiode:ComboDiode, F.Cu at (204.8, 119.9)
- moved D13 17.5 mm to (244.5, 62.7)
- moved D39 8.25 mm to (239.6, 108.0), turned to 0 degrees
- moved D40 7.53 mm to (259.6, 108.0), turned to 0 degrees
- moved D44 1.59 mm to (153.2, 119.9)
- moved D12 1.59 mm to (241.3, 62.7)
- moved D38 0.79 mm to (238.9, 100.8)
Routing:
- net (no net): track 0.00 -> 24.8 mm
- net COL5: track 123.5 -> 147.4 mm
- net COL8: track 181.1 -> 202.3 mm
- net COL9: track 197.6 -> 218.6 mm
- net COL4: track 97.7 -> 116.8 mm
- net COL12: track 268.3 -> 285.9 mm
- net COL13: track 284.3 -> 299.7 mm
- net Net-(D39-Pad2): track 14.3 -> 27.6 mm
- net Net-(D14-Pad2): track 20.3 -> 31.4 mm
- net Net-(D40-Pad2): track 13.1 -> 23.1 mm
- net Net-(D13-Pad2): track 7.51 -> 13.0 mm
- net ROW2: track 257.2 -> 261.0 mm
- net Net-(D38-Pad2): track 6.52 -> 9.26 mm
- net Net-(D12-Pad2): track 7.51 -> 5.72 mm
- net Net-(D44-Pad2): track 7.79 -> 6.54 mm
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Other:
- board text added: "V2.0"

Commit message: updating spacebars
Parts:
- removed the D1 at (134.1, 119.9)
- moved D44 19.0 mm to (134.1, 119.9)
Connections:
-   pad 1: COL5 -> COL6
-   pad 2: (no net) -> Net-(D44-Pad2)
Routing:
- net COL5: track 147.4 -> 123.5 mm
- net Net-(D44-Pad2): track 6.54 -> 24.3 mm
- net COL6: track 168.5 -> 183.5 mm
- net (no net): track 24.8 -> 18.9 mm
